Commit message: full model for gazebo with meshes

File: hexer_description/urdf/Hexer_v_1_0.urdf.xacro (robot description, xacro)
@@ -1,137 +1,145 @@
 <?xml version="1.0"?>
 <robot name="hexer_v_1_0" xmlns:xacro="http://www.ros.org/wiki/xacro">
-    <xacro:property name="radius_base" value="0.08" />
-    <xacro:property name="base_heigth" value="0.1" />
-    <xacro:property name="length_coxa" value="0.05" />
-    <xacro:property name="length_femur" value="0.07" />
-    <xacro:property name="length_tibia" value="0.27" />
-    <xacro:property name="radius_servo" value="0.021" />
-    <xacro:property name="leg_width" value="0.023" />
-    <xacro:property name="limit_servo_down" value="${-pi / 2.0}" />
-    <xacro:property name="limit_servo_up" value="${pi / 2.0}" />
-    <material name="grey">
-        <color rgba="0.5 0.5 0.5 1" />
-    </material>
-    <material name="coxa">
-        <color rgba="0.1 0.1 0.8 1" />
-    </material>
-    <material name="femur">
-        <color rgba="0.1 0.8 0.1 1" />
-    </material>
-    <material name="tibia">
-        <color rgba="0.8 0.1 0.1 1" />
-    </material>
-    <link name="base_link">
-        <visual>
-            <geometry>
-                <cylinder radius="${radius_base}" length="${base_heigth}" />
-            </geometry>
-            <origin xyz="0 0 0" rpy="0 0 0" />
-            <material name="grey" />
-        </visual>
-    </link>
+    <xacro:include filename="material.urdf.xacro" />
+    <xacro:include filename="base.urdf.xacro" />
     <link name="ground" />
     <joint name="ground_base_link" type="fixed">
-            <parent link="base_link" />
-            <child link="ground" />
-            <origin xyz="0 0 ${-(length_tibia - 0.1)}" rpy="0 0 0" />
+        <parent link="base_link" />
+        <child link="ground" />
+        <origin xyz="0 0 -0.225" rpy="0 0 0" />
     </joint>
-    <xacro:macro name="leg" params="prefix origin_x origin_y origin_z direction">
-        <link name="${prefix}_coxa_servo">
+    <xacro:macro name="leg_left" params="prefix origin_x origin_y origin_z">
+        <link name="${prefix}_coxa_left_link">
             <visual>
                 <geometry>
-                    <cylinder radius="${radius_servo}" length="${leg_width + (leg_width / 2.0)}" />
+                    <mesh filename="package://hexer_description/mesh/leg/coxa_left.stl" scale="0.001 0.001 0.001"/>
                 </geometry>
-                <origin xyz="0 0 0" rpy="0 0 0" />
+                <origin xyz="-0.0095 -0.02 -0.015" rpy="0 0 0" />
                 <material name="coxa" />
             </visual>
         </link>
-        <link name="${prefix}_coxa">
+        <link name="${prefix}_femur_left_link">
             <visual>
                 <geometry>
-                    <box size="${length_coxa} ${leg_width} ${leg_width}" />
+                    <mesh filename="package://hexer_description/mesh/leg/femur.stl" scale="0.001 0.001 0.001"/>
                 </geometry>
-                <origin xyz="0 0 0" rpy="0 0 0" />
+                <origin xyz="0 -0.035 -0.051" rpy="0 0 0" />
+                <material name="femur" />
+            </visual>
+        </link>
+        <link name="${prefix}_femur_left_two_link">
+            <visual>
+                <geometry>
+                    <mesh filename="package://hexer_description/mesh/leg/femur_two.stl" scale="0.001 0.001 0.001"/>
+                </geometry>
+                <origin xyz="-0.024 -0.01 -0.051" rpy="0 0 ${pi}" />
+                <material name="femur" />
+            </visual>
+        </link>
+        <link name="${prefix}_tibia_left_link">
+            <visual>
+                <geometry>
+                    <mesh filename="package://hexer_description/mesh/leg/tibia_right.stl" scale="0.001 0.001 0.001"/>
+                </geometry>
+                <origin xyz="0.01 -0.001 -0.0725" rpy="0 0 ${-pi / 2.0}" />
+                <material name="tibia" />
+            </visual>
+        </link>
+        <joint name="${prefix}_coxa_left_base" type="revolute">
+            <parent link="base_link" />
+            <child link="${prefix}_coxa_left_link" />
+            <origin xyz="${origin_x} ${origin_y} ${origin_z}" rpy="0 0 ${-pi / 2.0}" />
+            <axis xyz="0 0 1" />
+            <limit lower="${-pi / 2.0}" upper="${pi / 2.0}" velocity="100" effort="100" />
+        </joint>
+        <joint name="${prefix}_femur_left_coxa" type="revolute">
+            <parent link="${prefix}_coxa_left_link" />
+            <child link="${prefix}_femur_left_link" />
+            <origin xyz="-0.038 -0.0508 0.018" rpy="0 0 0" />
+            <axis xyz="1 0 0" />
+            <limit lower="${-pi / 2.0}" upper="${pi / 2.0}" velocity="100" effort="100" />
+        </joint>
+        <joint name="${prefix}_femur_left_two_femur" type="fixed">
+            <parent link="${prefix}_femur_left_link" />
+            <child link="${prefix}_femur_left_two_link" />
+            <origin xyz="0.065 0 0" rpy="0 0 0" />
+        </joint>
+        <joint name="${prefix}_tibia_left_femur" type="revolute">
+            <parent link="${prefix}_femur_left_link" />
+            <child link="${prefix}_tibia_left_link" />
+            <origin xyz="0.01 -0.07 0" rpy="0 0 0" />
+            <axis xyz="1 0 0" />
+            <limit lower="${-pi / 2.0}" upper="${pi / 2.0}" velocity="100" effort="100" />
+        </joint>
+    </xacro:macro>
+    <xacro:leg_left prefix="down"  origin_x="-0.04" origin_y="0.069" origin_z="-0.046" />
+    <xacro:leg_left prefix="mid"  origin_x="-0.08" origin_y="-0.001" origin_z="-0.046" />
+    <xacro:leg_left prefix="up"  origin_x="-0.04" origin_y="-0.069" origin_z="-0.046" />
+    <xacro:macro name="leg_right" params="prefix origin_x origin_y origin_z">
+        <link name="${prefix}_coxa_right_link">
+            <visual>
+                <geometry>
+                    <mesh filename="package://hexer_description/mesh/leg/coxa_right.stl" scale="0.001 0.001 0.001" />
+                </geometry>
+                <origin xyz="-0.067 0.0435 -0.0025" rpy="0 0 ${-pi / 2.0}" />
                 <material name="coxa" />
             </visual>
         </link>
-        <link name="${prefix}_femur_servo">
+        <link name="${prefix}_femur_right_link">
             <visual>
                 <geometry>
-                    <cylinder radius="${radius_servo}" length="${leg_width + (leg_width / 2.0)}" />
+                    <mesh filename="package://hexer_description/mesh/leg/femur.stl" scale="0.001 0.001 0.001"/>
                 </geometry>
-                <origin xyz="0 0 0" rpy="0 0 0" />
+                <origin xyz="0.035 0 -0.051" rpy="0 0 ${-pi / 2.0}" />
                 <material name="femur" />
             </visual>
         </link>
-        <link name="${prefix}_femur">
+        <link name="${prefix}_femur_right_two_link">
             <visual>
                 <geometry>
-                    <box size="${length_femur} ${leg_width} ${leg_width}" />
+                    <mesh filename="package://hexer_description/mesh/leg/femur_two.stl" scale="0.001 0.001 0.001"/>
                 </geometry>
-                <origin xyz="0 0 0" rpy="0 0 0" />
+                <origin xyz="0.06 0.023 -0.051" rpy="0 0 ${-3.0*pi / 2.0}" />
                 <material name="femur" />
             </visual>
         </link>
-        <link name="${prefix}_tibia_servo">
+        <link name="${prefix}_tibia_right_link">
             <visual>
                 <geometry>
-                    <cylinder radius="${radius_servo}" length="${leg_width + (leg_width / 2.0)}" />
+                    <mesh filename="package://hexer_description/mesh/leg/tibia_left.stl" scale="0.001 0.001 0.001"/>
                 </geometry>
-                <origin xyz="0 0 0" rpy="0 0 0" />
+                <origin xyz="0.003 -0.01875 -0.19525" rpy="0 0 ${pi}" />
                 <material name="tibia" />
             </visual>
         </link>
-        <link name="${prefix}_tibia">
-            <visual>
-                <geometry>
-                    <box size="${length_tibia} ${leg_width} ${leg_width}" />
-                </geometry>
-                <origin xyz="0 0 0" rpy="0 0 0" />
-                <material name="tibia" />
-            </visual>
-        </link>
-        <joint name="${prefix}_coxa_servo_base_joint" type="revolute">
+        <joint name="${prefix}_coxa_right_base" type="revolute">
             <parent link="base_link" />
-            <child link="${prefix}_coxa_servo" />
-            <origin xyz="${origin_x} ${origin_y} ${origin_z}" rpy="${direction} ${direction} ${pi / 2.0}" />
+            <child link="${prefix}_coxa_right_link" />
+            <origin xyz="${origin_x} ${origin_y} ${origin_z}" rpy="0 0 0" />
             <axis xyz="0 0 1" />
-            <limit lower="${limit_servo_down}" upper="${limit_servo_up}" velocity="100" effort="100" />
+            <limit lower="${-pi / 2.0}" upper="${pi / 2.0}" velocity="100" effort="100" />
         </joint>
-        <joint name="${prefix}_coxa_coxa_servo_joint" type="fixed">
-            <parent link="${prefix}_coxa_servo" />
-            <child link="${prefix}_coxa" />
-            <origin xyz="${length_coxa / 2.0} 0 0" rpy="0 0 0" />
+        <joint name="${prefix}_femur_right_coxa" type="revolute">
+            <parent link="${prefix}_coxa_right_link" />
+            <child link="${prefix}_femur_right_link" />
+            <origin xyz="0.0508 0.0385 0.018" rpy="0 0 0" />
+            <axis xyz="0 1 0" />
+            <limit lower="${-pi / 2.0}" upper="${pi / 2.0}" velocity="100" effort="100" />
         </joint>
-        <joint name="${prefix}_femur_servo_coxa" type="revolute">
-            <parent link="${prefix}_coxa" />
-            <child link="${prefix}_femur_servo" />
-            <origin xyz="${(length_coxa / 2.0)} 0 0" rpy="${pi / 2.0} 0 0" />
-            <axis xyz="0 0 1" />
-            <limit lower="${limit_servo_down}" upper="${limit_servo_up}" velocity="100" effort="100" />
+        <joint name="${prefix}_femur_right_two_femur" type="fixed">
+            <parent link="${prefix}_femur_right_link" />
+            <child link="${prefix}_femur_right_two_link" />
+            <origin xyz="0 -0.065 0" rpy="0 0 0" />
         </joint>
-        <joint name="${prefix}_femur_femur_servo_joint" type="fixed">
-            <parent link="${prefix}_femur_servo" />
-            <child link="${prefix}_femur" />
-            <origin xyz="${length_femur / 2.0} 0 0" rpy="0 0 0" />
-        </joint>
-        <joint name="${prefix}_tibia_servo_femur_joint" type="revolute">
-            <parent link="${prefix}_femur" />
-            <child link="${prefix}_tibia_servo" />
-            <origin xyz="${length_femur / 2.0} 0 0" rpy="0 0 0" />
-            <axis xyz="0 0 1" />
-            <limit lower="${limit_servo_down}" upper="${limit_servo_up}" velocity="100" effort="100" />
-        </joint>
-        <joint name="${prefix}_tibia_tibia_servo_joint" type="fixed">
-            <parent link="${prefix}_tibia_servo" />
-            <child link="${prefix}_tibia" />
-            <origin xyz="0 -0.035 0" rpy="0 0 ${pi/ 2.0}" />
+        <joint name="${prefix}_tibia_right_femur" type="revolute">
+            <parent link="${prefix}_femur_right_link" />
+            <child link="${prefix}_tibia_right_link" />
+            <origin xyz="0.07 -0.01 0" rpy="0 0 0" />
+            <axis xyz="0 1 0" />
+            <limit lower="${-pi / 2.0}" upper="${pi / 2.0}" velocity="100" effort="100" />
         </joint>
     </xacro:macro>
-    <xacro:leg prefix="right_up"  origin_x="0.07" origin_y="0.04" origin_z="0" direction="0" />
-    <xacro:leg prefix="right_mid" origin_x="0" origin_y="0.08" origin_z="0" direction="0"  />
-    <xacro:leg prefix="right_down" origin_x="-0.07" origin_y="0.04" origin_z="0" direction="0" />
-    <xacro:leg prefix="left_up" origin_x="0.07" origin_y="-0.04" origin_z="0"  direction="${pi}" />
-    <xacro:leg prefix="left_mid" origin_x="0" origin_y="-0.08" origin_z="0"  direction="${pi}" />
-    <xacro:leg prefix="left_down" origin_x="-0.07" origin_y="-0.04" origin_z="0"  direction="${pi}" />
+    <xacro:leg_right prefix="down" origin_x="0.04" origin_y="0.069" origin_z="-0.046" />
+    <xacro:leg_right prefix="mid" origin_x="0.08" origin_y="0" origin_z="-0.046" />
+    <xacro:leg_right prefix="up" origin_x="0.04" origin_y="-0.069" origin_z="-0.046" />
 </robot>

Commit message: inertia tags and collision update

File: hexer_description/urdf/Hexer_v_1_0.urdf.xacro (robot description, xacro)
@@ -1,11 +1,12 @@
 <?xml version="1.0"?>
 <robot name="hexer_v_1_0" xmlns:xacro="http://www.ros.org/wiki/xacro">
-    <xacro:include filename="material.urdf.xacro" />
+    <xacro:include filename="material.xacro" />
+    <xacro:include filename="inertia.xacro" />
     <xacro:include filename="base.urdf.xacro" />
     <link name="ground" />
     <joint name="ground_base_link" type="fixed">
-        <parent link="base_link" />
-        <child link="ground" />
-        <origin xyz="0 0 -0.225" rpy="0 0 0" />
+        <parent link="ground" />
+        <child link="base_link" />
+        <origin xyz="0 0 0.225" rpy="0 0 0" />
     </joint>
     <xacro:macro name="leg_left" params="prefix origin_x origin_y origin_z">
@@ -18,4 +19,11 @@
                 <material name="coxa" />
             </visual>
+            <collision>
+                <geometry>
+                    <box size="0.08 0.031 0.059" />
+                </geometry>
+                <origin xyz="-0.001 -0.0225 0.027" rpy="0 0 ${pi / 2.0}" />
+            </collision>
+            <xacro:coxa_inertia_left m="0.122" xyz="0 -0.03 0.02" rpy="0 0 0" />
         </link>
         <link name="${prefix}_femur_left_link">
@@ -27,4 +35,11 @@
                 <material name="femur" />
             </visual>
+            <collision>
+                <geometry>
+                    <box size="0.09 0.008 0.032" />
+                </geometry>
+                <origin xyz="0.005 -0.035 -0.0025" rpy="0 0 ${pi / 2.0}" />
+            </collision>
+            <xacro:femur_inertia_one_left m="0.013" xyz="0.005 -0.035 0" rpy="0 0 0" />
         </link>
         <link name="${prefix}_femur_left_two_link">
@@ -36,4 +51,11 @@
                 <material name="femur" />
             </visual>
+            <collision>
+                <geometry>
+                    <box size="0.09 0.008 0.032" />
+                </geometry>
+                <origin xyz="-0.00425 -0.035 -0.0025" rpy="0 0 ${pi / 2.0}" />
+            </collision>
+            <xacro:femur_inertia_one_left m="0.013" xyz="-0.005 -0.035 0" rpy="0 0 0" />
         </link>
         <link name="${prefix}_tibia_left_link">
@@ -45,4 +67,11 @@
                 <material name="tibia" />
             </visual>
+            <collision>
+                <geometry>
+                    <box size="0.025 0.025 0.275" />
+                </geometry>
+                <origin xyz="0.02 0.002 -0.055" rpy="0 0 ${pi / 2.0}" />
+            </collision>
+            <xacro:tibia_inertia_left m="0.12" xyz="0.02 0 -0.04" rpy="0 0 0" />
         </link>
         <joint name="${prefix}_coxa_left_base" type="revolute">
@@ -85,4 +114,11 @@
                 <material name="coxa" />
             </visual>
+            <collision>
+                <geometry>
+                    <box size="0.08 0.031 0.059" />
+                </geometry>
+                <origin xyz="0.0225 0 0.027" rpy="0 0 0" />
+            </collision>
+            <xacro:coxa_inertia_right m="0.122" xyz="0.03 0 0.02" rpy="0 0 0" />
         </link>
         <link name="${prefix}_femur_right_link">
@@ -94,4 +130,11 @@
                 <material name="femur" />
             </visual>
+            <collision>
+                <geometry>
+                    <box size="0.09 0.008 0.032" />
+                </geometry>
+                <origin xyz="0.035 -0.005 -0.0025" rpy="0 0 0" />
+            </collision>
+            <xacro:femur_inertia_one_right m="0.013" xyz="0.035 -0.005 0" rpy="0 0 0" />
         </link>
         <link name="${prefix}_femur_right_two_link">
@@ -103,4 +146,11 @@
                 <material name="femur" />
             </visual>
+            <collision>
+                <geometry>
+                    <box size="0.09 0.008 0.032" />
+                </geometry>
+                <origin xyz="0.035 0.00325 -0.0025" rpy="0 0 0" />
+            </collision>
+            <xacro:femur_inertia_one_right m="0.013" xyz="0.035 0.005 0" rpy="0 0 0" />
         </link>
         <link name="${prefix}_tibia_right_link">
@@ -112,4 +162,11 @@
                 <material name="tibia" />
             </visual>
+            <collision>
+                <geometry>
+                    <box size="0.025 0.025 0.275" />
+                </geometry>
+                <origin xyz="-0.002 -0.02 -0.055" rpy="0 0 ${pi / 2.0}" />
+            </collision>
+            <xacro:tibia_inertia_right m="0.12" xyz="0 -0.02 -0.04" rpy="0 0 0" />
         </link>
         <joint name="${prefix}_coxa_right_base" type="revolute">

File: hexer_description/urdf/base.urdf.xacro (robot description, xacro)
@@ -9,4 +9,11 @@
             <material name="black" />
         </visual>
+        <collision>
+            <geometry>
+                <box size="0.14 0.16 0.012" />
+            </geometry>
+            <origin xyz="0 0 0.011" rpy="0 0 0" />
+        </collision>
+        <xacro:main_body_inertia m="0.094" xyz="0 0 0" rpy="0 0 0" />
     </link>
     <link name="base_down_link">
@@ -18,4 +25,11 @@
             <material name="black" />
         </visual>
+        <collision>
+            <geometry>
+                <box size="0.14 0.16 0.012" />
+            </geometry>
+            <origin xyz="0 0 0.011" rpy="0 0 0" />
+        </collision>
+        <xacro:main_body_down_inertia m="0.066" xyz="0 0 0" rpy="0 0 0" />
     </link>
     <link name="base_up_link">
@@ -27,4 +41,11 @@
             <material name="black" />
         </visual>
+        <collision>
+            <geometry>
+                <box size="0.14 0.16 0.012" />
+            </geometry>
+            <origin xyz="0 0 0.031" rpy="0 0 0" />
+        </collision>
+        <xacro:main_body_up_inertia m="0.135" xyz="0 0 0" rpy="0 0 0" />
     </link>
     <joint name="down_base_link" type="fixed">
